File: TinyLoRa-Breakout/TLM-breakout-v1/TLM-breakout-v1.sch (KiCad schematic (older format))
At the start: 45 parts, among them J1 SMA-Edge-Mount, J2 U.FL-R-SMT-1, J3 JST_PH, J4 USB_B_Micro, J5 Cortex_JTAG_SWD_10pin, SW3 RESET, U1 TLM01, U2 MCP73831-2-OT, U3 TPS3839DBZ, U4 S-1313C33, U5 NUP2114, U6 Feather-Generic

Commit message: BOMs added
BOMs for TinyLoRa and its breakout added
Parts:
- C1, C2, C3, C4, C5, C6, C7, C8, C9, D2, D3, JP2, JP3, JP4, JP5, L1, R1, R10, R11, R12, R2, R3, R4, R5, R6, R7, R8, R9, U1, U6: Mfg (none) -> -
- D1: Mfg (none) -> MBR120VLSFT3G
- D4: value LED_PWR -> LED_PWR_BLUE; Mfg (none) -> -
- D5: value LED0 -> LED0_RED; Mfg (none) -> -
- F1: Mfg (none) -> MF-PSMF075X-2
- J1: Mfg (none) -> SMA-J-P-H-ST-EM1
- J2: Mfg (none) -> U.FL-R-SMT-1(40)
- J3: Mfg S2B-PH-K-S(LF) -> S2B-PH-SM4-TB(LF)(SN)
- J4: Mfg (none) -> 629105150521
- J5: Mfg (none) -> FTSH-105-01-F-DV-K
- SW3: Mfg (none) -> EVQ-P2202M
- U2: value MCP73831-2-OT -> MCP73831; Mfg (none) -> MCP73831T-2ATI/OT
- U3: Mfg (none) -> TPS3839G33DBZR
- U4: Mfg (none) -> S-1313C33-M5T1U3
- U5: Mfg (none) -> NUP2114UPXV5T1G
Changed lines of the file:
@@
 F 2 "TLM-footprints:TLM-01-footprint" H 8250 1750 39  0001 C CNN
 F 3 "" H 8250 1750 39  0001 C CNN
+F 4 "-" H 0   0   50  0001 C CNN "Mfg"
 	1    8200 1700
 	1    0    0    -1
@@
 F 2 "mySMA_Connectos:SMA_J_P_X_ST_EM1_EdgeMount" H 9475 1025 50  0001 C CNN
 F 3 " ~" H 9475 1025 50  0001 C CNN
+F 4 "SMA-J-P-H-ST-EM1 " H 0   0   50  0001 C CNN "Mfg"
 	1    9475 1025
 	1    0    0    -1
@@
 F 2 "Connector_USB:USB_Micro-B_Wuerth_629105150521" H 1725 3325 50  0001 C CNN
 F 3 "~" H 1725 3325 50  0001 C CNN
+F 4 "629105150521 " H 0   0   50  0001 C CNN "Mfg"
 	1    1575 3375
 	1    0    0    -1
@@
 F 2 "Package_TO_SOT_SMD:SOT-23-5" H 5325 1800 50  0001 C CIN
 F 3 "http://www.ti.com/lit/ds/symlink/tlv702.pdf" H 5325 1525 50  0001 C CNN
+F 4 "S-1313C33-M5T1U3 " H 0   0   50  0001 C CNN "Mfg"
 	1    5325 1475
 	1    0    0    -1
@@
 F 2 "Package_TO_SOT_SMD:SOT-23" H 4025 1475 50  0001 C CNN
 F 3 "http://www.ti.com/lit/ds/sbvs193d/sbvs193d.pdf" H 4025 1475 50  0001 C CNN
+F 4 "TPS3839G33DBZR " H 0   0   50  0001 C CNN "Mfg"
 	1    4025 1475
 	1    0    0    -1
@@
 F 2 "Connector_JST:JST_PH_S2B-PH-SM4-TB_1x02-1MP_P2.00mm_Horizontal" H 800 1100 50  0001 C CNN
 F 3 "~" H 800 1100 50  0001 C CNN
-F 4 "S2B-PH-K-S(LF)" H 800 1100 50  0001 C CNN "Mfg"
+F 4 "S2B-PH-SM4-TB(LF)(SN) " H 800 1100 50  0001 C CNN "Mfg"
 	1    800  1100
 	-1   0    0    -1
@@
 F 2 "Diode_SMD:D_SOD-123" H 4625 925 50  0001 C CNN
 F 3 "http://www.mccsemi.com/up_pdf/MBR0520~MBR0580(SOD123).pdf" H 4625 1100 50  0001 C CNN
+F 4 "MBR120VLSFT3G" H 0   0   50  0001 C CNN "Mfg"
 	1    4625 1100
 	0    -1   -1   0
@@
 P 2300 1300
 F 0 "U2" H 2025 1550 50  0000 C CNN
-F 1 "MCP73831-2-OT" H 2675 1550 50  0000 C CNN
+F 1 "MCP73831" H 2675 1550 50  0000 C CNN
 F 2 "Package_TO_SOT_SMD:SOT-23-5" H 2350 1050 50  0001 L CIN
 F 3 "http://ww1.microchip.com/downloads/en/DeviceDoc/20001984g.pdf" H 2150 1250 50  0001 C CNN
+F 4 "MCP73831T-2ATI/OT " H 0   0   50  0001 C CNN "Mfg"
 	1    2300 1300
 	1    0    0    -1
@@
 F 2 "Resistor_SMD:R_0402_1005Metric" V 1405 4050 50  0001 C CNN
 F 3 "~" H 1475 4050 50  0001 C CNN
+F 4 "-" H 0   0   50  0001 C CNN "Mfg"
 	1    1475 4050
 	1    0    0    1
@@
 F 2 "Capacitor_SMD:C_0603_1608Metric" H 1213 3900 50  0001 C CNN
 F 3 "~" H 1175 4050 50  0001 C CNN
+F 4 "-" H 0   0   50  0001 C CNN "Mfg"
 	1    1175 4050
 	1    0    0    1
@@
 F 2 "Capacitor_SMD:C_0603_1608Metric" H 2388 2700 50  0001 C CNN
 F 3 "~" H 2350 2850 50  0001 C CNN
+F 4 "-" H 0   0   50  0001 C CNN "Mfg"
 	1    2350 2850
 	1    0    0    -1
@@
 F 2 "Fuse:Fuse_0805_2012Metric" H 3125 2475 50  0001 L CNN
 F 3 "~" H 3075 2675 50  0001 C CNN
+F 4 "MF-PSMF075X-2" H 0   0   50  0001 C CNN "Mfg"
 	1    3075 2675
 	0    -1   -1   0
@@
 F 2 "Capacitor_SMD:C_0603_1608Metric" H 2888 2700 50  0001 C CNN
 F 3 "~" H 2850 2850 50  0001 C CNN
+F 4 "-" H 0   0   50  0001 C CNN "Mfg"
 	1    2850 2850
 	1    0    0    -1
@@
 F 2 "Connector_PinHeader_1.27mm:PinHeader_2x05_P1.27mm_Vertical_SMD" H 1950 4900 50  0001 L TNN
 F 3 "http://infocenter.arm.com/help/topic/com.arm.doc.faqs/attached/13634/cortex_debug_connectors.pdf" V 1550 4200 50  0001 C CNN
+F 4 "FTSH-105-01-F-DV-K " H 0   0   50  0001 C CNN "Mfg"
 	1    1900 5450
 	1    0    0    -1
@@
 P 4625 3575
 F 0 "D5" V 4663 3457 50  0000 R CNN
-F 1 "LED0" V 4572 3457 50  0000 R CNN
+F 1 "LED0_RED" V 4572 3457 50  0000 R CNN
 F 2 "LED_SMD:LED_0603_1608Metric" H 4625 3575 50  0001 C CNN
 F 3 "~" H 4625 3575 50  0001 C CNN
+F 4 "-" H 0   0   50  0001 C CNN "Mfg"
 	1    4625 3575
 	0    -1   -1   0
@@
 F 2 "Jumper:SolderJumper-2_P1.3mm_Bridged_RoundedPad1.0x1.5mm" H 4625 3225 50  0001 C CNN
 F 3 "~" H 4625 3225 50  0001 C CNN
+F 4 "-" H 0   0   50  0001 C CNN "Mfg"
 	1    4625 3225
 	0    1    1    0
@@
 F 2 "Resistor_SMD:R_0402_1005Metric" V 4555 3925 50  0001 C CNN
 F 3 "~" H 4625 3925 50  0001 C CNN
+F 4 "-" H 0   0   50  0001 C CNN "Mfg"
 	1    4625 3925
 	-1   0    0    -1
@@
 F 2 "Capacitor_SMD:C_0603_1608Metric" H 4663 1500 50  0001 C CNN
 F 3 "~" H 4625 1650 50  0001 C CNN
+F 4 "-" H 0   0   50  0001 C CNN "Mfg"
 	1    4625 1650
 	1    0    0    -1
@@
 F 2 "Capacitor_SMD:C_0603_1608Metric" H 5838 1500 50  0001 C CNN
 F 3 "~" H 5800 1650 50  0001 C CNN
+F 4 "-" H 0   0   50  0001 C CNN "Mfg"
 	1    5800 1650
 	1    0    0    -1
@@
 F 2 "Capacitor_SMD:C_0603_1608Metric" H 6188 1500 50  0001 C CNN
 F 3 "~" H 6150 1650 50  0001 C CNN
+F 4 "-" H 0   0   50  0001 C CNN "Mfg"
 	1    6150 1650
 	1    0    0    -1
@@
 P 4325 3575
 F 0 "D4" V 4350 3750 50  0000 R CNN
-F 1 "LED_PWR" V 4250 3975 50  0000 R CNN
+F 1 "LED_PWR_BLUE" V 4250 3975 50  0000 R CNN
 F 2 "LED_SMD:LED_0603_1608Metric" H 4325 3575 50  0001 C CNN
 F 3 "~" H 4325 3575 50  0001 C CNN
+F 4 "-" H 0   0   50  0001 C CNN "Mfg"
 	1    4325 3575
 	0    -1   -1   0
@@
 F 2 "Jumper:SolderJumper-2_P1.3mm_Bridged_RoundedPad1.0x1.5mm" H 4325 3225 50  0001 C CNN
 F 3 "~" H 4325 3225 50  0001 C CNN
+F 4 "-" H 0   0   50  0001 C CNN "Mfg"
 	1    4325 3225
 	0    -1   1    0
@@
 F 2 "Resistor_SMD:R_0402_1005Metric" V 4255 3925 50  0001 C CNN
 F 3 "~" H 4325 3925 50  0001 C CNN
+F 4 "-" H 0   0   50  0001 C CNN "Mfg"
 	1    4325 3925
 	1    0    0    -1
@@
 F 2 "LED_SMD:LED_0603_1608Metric" H 3275 1400 50  0001 C CNN
 F 3 "~" H 3275 1400 50  0001 C CNN
+F 4 "-" H 0   0   50  0001 C CNN "Mfg"
 	1    3275 1400
 	1    0    0    1
@@
 F 2 "LED_SMD:LED_0603_1608Metric" H 3275 1575 50  0001 C CNN
 F 3 "~" H 3275 1575 50  0001 C CNN
+F 4 "-" H 0   0   50  0001 C CNN "Mfg"
 	1    3275 1575
 	-1   0    0    1
@@
 F 2 "Capacitor_SMD:C_0603_1608Metric" H 2913 1500 50  0001 C CNN
 F 3 "~" H 2875 1650 50  0001 C CNN
+F 4 "-" H 0   0   50  0001 C CNN "Mfg"
 	1    2875 1650
 	1    0    0    1
@@
 F 2 "Resistor_SMD:R_0402_1005Metric" V 1755 1625 50  0001 C CNN
 F 3 "~" H 1825 1625 50  0001 C CNN
+F 4 "-" H 0   0   50  0001 C CNN "Mfg"
 	1    1825 1625
 	-1   0    0    -1
@@
 F 2 "Resistor_SMD:R_0402_1005Metric" H 4750 1475 50  0001 C CNN
 F 3 "~" H 4750 1475 50  0001 C CNN
+F 4 "-" H 0   0   50  0001 C CNN "Mfg"
 	1    4750 1475
 	0    1    1    0
@@
 F 2 "Inductor_SMD:L_0402_1005Metric" H 8150 1025 50  0001 C CNN
 F 3 "~" H 8150 1025 50  0001 C CNN
+F 4 "-" H 0   0   50  0001 C CNN "Mfg"
 	1    8150 1025
 	0    -1   -1   0
@@
 F 2 "Capacitor_SMD:C_0402_1005Metric" H 8325 1150 50  0001 C CNN
 F 3 "~" H 8325 1150 50  0001 C CNN
+F 4 "-" H 0   0   50  0001 C CNN "Mfg"
 	1    8325 1150
 	-1   0    0    -1
@@
 F 2 "Resistor_SMD:R_0402_1005Metric" H 8750 1025 50  0001 C CNN
 F 3 "~" H 8750 1025 50  0001 C CNN
+F 4 "-" H 0   0   50  0001 C CNN "Mfg"
 	1    8750 1025
 	0    1    1    0
@@
 F 2 "Resistor_SMD:R_0402_1005Metric" H 9050 1025 50  0001 C CNN
 F 3 "~" H 9050 1025 50  0001 C CNN
+F 4 "-" H 0   0   50  0001 C CNN "Mfg"
 	1    9050 1025
 	0    1    1    0
@@
 F 2 "Resistor_SMD:R_0402_1005Metric" V 6055 5575 50  0001 C CNN
 F 3 "~" H 6125 5575 50  0001 C CNN
+F 4 "-" H 0   0   50  0001 C CNN "Mfg"
 	1    6125 5575
 	-1   0    0    1
@@
 F 2 "Resistor_SMD:R_0402_1005Metric" V 6055 5975 50  0001 C CNN
 F 3 "~" H 6125 5975 50  0001 C CNN
+F 4 "-" H 0   0   50  0001 C CNN "Mfg"
 	1    6125 5975
 	-1   0    0    1
@@
 F 2 "Capacitor_SMD:C_0603_1608Metric" H 5863 5825 50  0001 C CNN
 F 3 "~" H 5825 5975 50  0001 C CNN
+F 4 "-" H 0   0   50  0001 C CNN "Mfg"
 	1    5825 5975
 	1    0    0    1
@@
 F 2 "Jumper:SolderJumper-2_P1.3mm_Bridged_RoundedPad1.0x1.5mm" H 5675 5575 50  0001 C CNN
 F 3 "~" H 5675 5575 50  0001 C CNN
+F 4 "-" H 0   0   50  0001 C CNN "Mfg"
 	1    5675 5575
 	0    1    1    0
@@
 F 2 "Connector_Coaxial:U.FL_Hirose_U.FL-R-SMT-1_Vertical" H 7800 1025 50  0001 C CNN
 F 3 " ~" H 7800 1025 50  0001 C CNN
+F 4 "U.FL-R-SMT-1(40) " H 0   0   50  0001 C CNN "Mfg"
 	1    7800 1025
 	-1   0    0    -1
@@
 F 2 "Button_Switch_SMD:SW_SPST_EVQP2" H 5800 4000 50  0001 C CNN
 F 3 "" H 5800 4000 50  0001 C CNN
+F 4 " EVQ-P2202M " H 0   0   50  0001 C CNN "Mfg"
 	1    5800 3800
 	0    -1   -1   0
@@
 F 2 "Resistor_SMD:R_0402_1005Metric" V 5730 3400 50  0001 C CNN
 F 3 "~" H 5800 3400 50  0001 C CNN
+F 4 "-" H 0   0   50  0001 C CNN "Mfg"
 	1    5800 3400
 	-1   0    0    -1
@@
 F 2 "Package_TO_SOT_SMD:SOT-553" H 2375 4500 50  0001 C CNN
 F 3 "http://www.onsemi.ru.com/pub_link/Collateral/NUP2202W1-D.PDF" H 2255 4075 50  0001 C CNN
+F 4 "NUP2114UPXV5T1G " H 0   0   50  0001 C CNN "Mfg"
 	1    2175 4000
 	1    0    0    -1
@@
 F 2 "Jumper:SolderJumper-2_P1.3mm_Bridged_RoundedPad1.0x1.5mm" H 6125 5200 50  0001 C CNN
 F 3 "~" H 6125 5200 50  0001 C CNN
+F 4 "-" H 0   0   50  0001 C CNN "Mfg"
 	1    6125 5200
 	0    -1   1    0
@@
 F 2 "mcu_footprints:Feather-Generic" H 8525 4450 50  0001 C CNN
 F 3 "" H 8525 4450 50  0001 C CNN
+F 4 "-" H 0   0   50  0001 C CNN "Mfg"
 	1    8525 4450
 	1    0    0    -1
@@
 F 2 "Resistor_SMD:R_0402_1005Metric" V 3405 1050 50  0001 C CNN
 F 3 "~" H 3475 1050 50  0001 C CNN
+F 4 "-" H 0   0   50  0001 C CNN "Mfg"
 	1    3475 1050
 	-1   0    0    -1
@@
 F 2 "Resistor_SMD:R_0402_1005Metric" V 3405 1725 50  0001 C CNN
 F 3 "~" H 3475 1725 50  0001 C CNN
+F 4 "-" H 0   0   50  0001 C CNN "Mfg"
 	1    3475 1725
 	-1   0    0    -1
