File: TinyLoRa-RF-Module/TLM-v1.2/TLM-v1_2.sch (KiCad schematic (older format))
At the start: 54 parts, among them U1 TLM01, U2 ATSAMR34J18B, U3 SKY13373-460LF, Y1 ABS05-32.768KHZ-9-T

Commit message: Minor changes
Other:
- note removed: "TCXO Default VCC \nfor the RF Switch"
Changed lines of the file:
@@
 EESchema Schematic File Version 4
 LIBS:TLM-v1_2-cache
-EELAYER 29 0
+EELAYER 30 0
 EELAYER END
 $Descr A4 11693 8268
@@
 Text GLabel 9825 5900 2    59   Input ~ 12
 TCXO_PWR
+Wire Wire Line
+	9025 5575 9400 5575
+Wire Wire Line
+	9025 5100 9025 5575
+Wire Wire Line
+	9400 5600 9400 5575
+Connection ~ 9400 5575
+Wire Wire Line
+	9400 5575 9675 5575
+Wire Wire Line
+	9825 5775 9825 5900
+$Comp
+L power:VDDA #PWR044
+U 1 1 5C5A5F40
+P 9825 5350
+F 0 "#PWR044" H 9825 5200 50  0001 C CNN
+F 1 "VDDA" H 9825 5500 50  0000 C CNB
+F 2 "" H 9825 5350 50  0001 C CNN
+F 3 "" H 9825 5350 50  0001 C CNN
+	1    9825 5350
+	1    0    0    -1
+$EndComp
+Wire Wire Line
+	9825 5350 9825 5375
+$Comp
+L power:GND #PWR?
+U 1 1 5D43B50A
+P 9250 4075
+F 0 "#PWR?" H 9250 3825 50  0001 C CNN
+F 1 "GND" H 9255 3902 50  0000 C CNN
+F 2 "" H 9250 4075 50  0001 C CNN
+F 3 "" H 9250 4075 50  0001 C CNN
+	1    9250 4075
+	1    0    0    -1
+$EndComp
+Wire Wire Line
+	9250 4075 9075 4075
+Text GLabel 8700 5475 0    59   Input ~ 12
+TXRX_RF
 $Comp
 L Jumper:SolderJumper_3_Bridged12 JP1
@@
 	0    1    -1   0
 $EndComp
-Wire Wire Line
-	9025 5575 9400 5575
-Wire Wire Line
-	9025 5100 9025 5575
-Wire Wire Line
-	9400 5600 9400 5575
-Connection ~ 9400 5575
-Wire Wire Line
-	9400 5575 9675 5575
-Wire Wire Line
-	9825 5775 9825 5900
-$Comp
-L power:VDDA #PWR044
-U 1 1 5C5A5F40
-P 9825 5350
-F 0 "#PWR044" H 9825 5200 50  0001 C CNN
-F 1 "VDDA" H 9825 5500 50  0000 C CNB
-F 2 "" H 9825 5350 50  0001 C CNN
-F 3 "" H 9825 5350 50  0001 C CNN
-	1    9825 5350
-	1    0    0    -1
-$EndComp
-Wire Wire Line
-	9825 5350 9825 5375
-$Comp
-L power:GND #PWR?
-U 1 1 5D43B50A
-P 9250 4075
-F 0 "#PWR?" H 9250 3825 50  0001 C CNN
-F 1 "GND" H 9255 3902 50  0000 C CNN
-F 2 "" H 9250 4075 50  0001 C CNN
-F 3 "" H 9250 4075 50  0001 C CNN
-	1    9250 4075
-	1    0    0    -1
-$EndComp
-Wire Wire Line
-	9250 4075 9075 4075
-Text GLabel 8700 5475 0    59   Input ~ 12
-TXRX_RF
-Text Notes 9850 6225 0    59   ~ 12
-TCXO Default VCC \nfor the RF Switch
-Wire Notes Line
-	9575 6300 10925 6300
-Wire Notes Line
-	10925 6300 10925 5975
-Wire Notes Line
-	10925 5975 9575 5975
-Wire Notes Line
-	9575 5975 9575 6300
 $EndSCHEMATC
