File: TinyLoRa-Feather-Breakout/TinyLoRa-Feather-4260-v1_0/TinyLoRa-Feather-4260-v1_0.sch (KiCad schematic (older format))
At the start: 57 parts, among them J1 U.FL-R-SMT-1, J2 SMA-Edge-Mount, J3 USB_C_Receptacle_USB2.0, J4 JST_PH, J5 Conn_ARM_JTAG_SWD_10, Q1 SI2323DS, SW1 USR_BTN, SW2 RESET, U1 MCP73831, U2 ME6215C33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

Commit message: Naming updates
Parts:
- D5: symbol TLM-4260-breakout-v1_0-rescue:RGB_LED_FM-B2020RGBA-tinylora_v1 -> TinyLoRa-Feather-4260-v1_0-rescue:RGB_LED_FM-B2020RGBA-tinylora_v1-TLM-4260-breakout-v1_0-rescue-TinyLoRa-4260-breakout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
- U4: symbol TLM-4260-breakout-v1_0-rescue:RAK4260-rak4260 -> TinyLoRa-Feather-4260-v1_0-rescue:RAK4260-rak4260-TLM-4260-breakout-v1_0-rescue-TinyLoRa-4260-breakout-v1_0-rescue
- U6: symbol TLM-4260-breakout-v1_0-rescue:Feather-Generic-my-Arduino-Boards -> TinyLoRa-Feather-4260-v1_0-rescue:Feather-Generic-my-Arduino-Boards-TLM-4260-breakout-v1_0-rescue-TinyLoRa-4260-breakou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
- U7: symbol TLM-4260-breakout-v1_0-rescue:ATECC608A-SSHDA-Security -> TinyLoRa-Feather-4260-v1_0-rescue:ATECC608A-SSHDA-Security-TLM-4260-breakout-v1_0-rescue-TinyLoRa-4260-breakout-v1_0-re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
Other:
- note added: "BAND_SEL\nRFSW VCC\nTCXO PWR"
- note added: "PA13\nPA09\nPA09"
- note added: "PA13\nPA28\nPB03"
- note added: "RAK4260 TLM01-v1.2\n"
- note added: "SAMR34 Pins which are NC/used internally:"
- note removed: "~Notes:\nSAMR34 Pins which are NC/used internally.\n- PA13 (BAND_SEL*)\n- PA28 (TCXO PWR*)\n- PB03 (Backup Bat)\n\n*to be verified"
Changed lines of the file:
@@
 EESchema Schematic File Version 4
-LIBS:TLM-4260-breakout-v1_0-cache
+LIBS:TinyLoRa-Feather-4260-v1_0-cache
 EELAYER 30 0
 EELAYER END
@@
 encoding utf-8
 Sheet 1 1
-Title "TinyLoRa RAK4260 Feather Breakout"
+Title "TinyLoRa Feather RAK4260 Breakout"
 Date "2019-11-04"
 Rev "1.0"
@@
 Wire Notes Line
 	11175 500  6550 500
-Text Notes 6625 4175 0    59   Italic 12
+Text Notes 9125 4175 0    59   Italic 12
 RAK4260 ATSAMR34 based RF+MCU Module
 $Comp
@@
 $EndComp
 $Comp
-L TLM-4260-breakout-v1_0-rescue:Feather-Generic-my-Arduino-Boards U6
+L TinyLoRa-Feather-4260-v1_0-rescue:Feather-Generic-my-Arduino-Boards-TLM-4260-breakout-v1_0-rescue-TinyLoRa-4260-breakout-v1_0-rescue U6
 U 1 1 5DC21E0A
 P 8450 4650
@@
 90 Ω diff trace
 $Comp
-L TLM-4260-breakout-v1_0-rescue:RAK4260-rak4260 U4
+L TinyLoRa-Feather-4260-v1_0-rescue:RAK4260-rak4260-TLM-4260-breakout-v1_0-rescue-TinyLoRa-4260-breakout-v1_0-rescue U4
 U 1 1 5DE73C41
 P 8750 2100
@@
 Wire Wire Line
 	5575 5750 5650 5750
-Text Notes 6625 3950 0    59   Italic 0
-~Notes:\nSAMR34 Pins which are NC/used internally.\n- PA13 (BAND_SEL*)\n- PA28 (TCXO PWR*)\n- PB03 (Backup Bat)\n\n*to be verified
+Text Notes 6650 4050 0    59   Italic 0
+SAMR34 Pins which are NC/used internally:
 Text Notes 10650 2725 0    50   ~ 0
 PA28
@@
 Pre-Provisioned secure element \nwith LoRaWAN TTN Join Server \nSOIC-8 (Optional)
 $Comp
-L TLM-4260-breakout-v1_0-rescue:ATECC608A-SSHDA-Security U7
+L TinyLoRa-Feather-4260-v1_0-rescue:ATECC608A-SSHDA-Security-TLM-4260-breakout-v1_0-rescue-TinyLoRa-4260-breakout-v1_0-rescue U7
 U 1 1 5EAF211B
 P 4875 5450
@@
 	475  4575 6525 4575
 $Comp
-L TLM-4260-breakout-v1_0-rescue:RGB_LED_FM-B2020RGBA-tinylora_v1 D5
+L TinyLoRa-Feather-4260-v1_0-rescue:RGB_LED_FM-B2020RGBA-tinylora_v1-TLM-4260-breakout-v1_0-rescue-TinyLoRa-4260-breakout-v1_0-rescue D5
 U 1 1 5DC3BE6D
 P 4800 3325
@@
 Text GLabel 5750 2475 0    39   BiDi ~ 8
 PA15
+Text Notes 6675 3925 0    50   ~ 10
+BAND_SEL\nRFSW VCC\nTCXO PWR
+Text Notes 7225 3925 0    50   ~ 0
+PA13\nPA28\nPB03
+Text Notes 7750 3925 0    50   ~ 0
+PA13\nPA09\nPA09
+Text Notes 7150 3650 0    50   ~ 10
+RAK4260    TLM01-v1.2\n
+Wire Notes Line
+	6675 3650 8125 3650
+Wire Notes Line
+	7575 3600 7575 3950
+Wire Notes Line
+	7100 3600 7100 3950
 $EndSCHEMATC
