File: Penguino-Hardware/Penguino-Feather-4260-v1_0/Penguino-Feather-4260-v1_0.sch (KiCad schematic (older format))
At the start: 57 parts, among them J1 U.FL-R-SMT-1, J2 SMA-Edge-Mount, J3 USB_C_Receptacle_USB2.0, J4 JST_PH, J5 Conn_ARM_JTAG_SWD_10, Q1 SI2323DS, SW1 USR_BTN, SW2 RESET, U1 MCP73831, U2 ME6215C33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

Commit message: Name changes
Parts:
- D5: symbol TinyLoRa-Feather-4260-v1_0-rescue:RGB_LED_FM-B2020RGBA-tinylora_v1-TLM-4260-breakout-v1_0-rescue-TinyLoRa-4260-breakout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 -> Penguino-Feather-4260-v1_0-rescue:RGB_LED_FM-B2020RGBA-tinylora_v1-TLM-4260-breakout-v1_0-rescue-TinyLoRa-4260-breakout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
- U2: symbol Regulator_Linear:TLV70233_SOT23-5 -> Penguino-Feather-4260-v1_0-rescue:TLV70233_SOT23-5-Regulator_Linear-TinyLoRa-Feather-4260-v1_0-rescue-Penguino-Feather-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
- U4: symbol TinyLoRa-Feather-4260-v1_0-rescue:RAK4260-rak4260-TLM-4260-breakout-v1_0-rescue-TinyLoRa-4260-breakout-v1_0-rescue -> Penguino-Feather-4260-v1_0-rescue:RAK4260-rak4260-TLM-4260-breakout-v1_0-rescue-TinyLoRa-4260-breakout-v1_0-rescue-Tiny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
- U6: symbol TinyLoRa-Feather-4260-v1_0-rescue:Feather-Generic-my-Arduino-Boards-TLM-4260-breakout-v1_0-rescue-TinyLoRa-4260-breakou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 -> Penguino-Feather-4260-v1_0-rescue:Feather-Generic-my-Arduino-Boards-TLM-4260-breakout-v1_0-rescue-TinyLoRa-4260-breakou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
- U7: symbol TinyLoRa-Feather-4260-v1_0-rescue:ATECC608A-SSHDA-Security-TLM-4260-breakout-v1_0-rescue-TinyLoRa-4260-breakout-v1_0-re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 -> Penguino-Feather-4260-v1_0-rescue:ATECC608A-SSHDA-Security-TLM-4260-breakout-v1_0-rescue-TinyLoRa-4260-breakout-v1_0-re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
Other:
- moved on the sheet: J4
