File: Penguino-Hardware/Penguino-Feather-4260-v1/Penguino-Feather-4260-v1.sch (KiCad schematic (older format))
At the start: 57 parts, among them J1 U.FL-R-SMT-1, J2 SMA-Edge-Mount, J3 USB_C_Receptacle_USB2.0, J4 JST_PH, J5 Conn_ARM_JTAG_SWD_10, Q1 SI2323DS, SW1 USR_BTN, SW2 RESET, U1 MCP73831, U2 ME6215C33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

Commit message: RAK4260 datasheet pin error
PA19 and PA18 are swapped
Parts:
- removed U4: RAK4260, rak4260:RAK4260-footprint_w_solder_paste, symbol Penguino-Feather-4260-v1-rescue:RAK4260-rak4260-TLM-4260-breakout-v1_0-rescue-T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
- added U4: RAK4260, rak4260:RAK4260-footprint_w_solder_paste, symbol rak4260:RAK4260
Other:
- note removed: "PA28"
Changed lines of the file:
@@
 90 Ω diff trace
-$Comp
-L Penguino-Feather-4260-v1-rescue:RAK4260-rak4260-TLM-4260-breakout-v1_0-rescue-TinyLoRa-4260-breakout-v1_0-rescue-TinyLoRa-Feather-4260-v1_0-rescue-Penguino-Feather-4260-v1_0-rescue-Penguino-Feather-4260-v1_0-rescue U4
-U 1 1 5DE73C41
-P 8750 2100
-F 0 "U4" H 8725 2675 59  0000 L CNB
-F 1 "RAK4260" H 9350 1750 79  0000 L CNB
-F 2 "rak4260:RAK4260-footprint_w_solder_paste" H 8650 2100 50  0001 C CNN
-F 3 "" H 8650 2100 50  0001 C CNN
-	1    8750 2100
-	1    0    0    -1
-$EndComp
 $Comp
 L Device:C_Small C5
@@
 Wire Wire Line
 	9550 3400 9550 4000
+Text GLabel 10650 2800 2    39   BiDi ~ 8
+PA18_TX3
 Text GLabel 10650 2900 2    39   BiDi ~ 8
-PA18_TX3
-Text GLabel 10650 2800 2    39   BiDi ~ 8
 PA19_RX3
 Wire Wire Line
@@
 Text Notes 6650 4050 0    59   Italic 0
 SAMR34 Pins which are NC/used internally:
-Text Notes 10650 2725 0    50   ~ 0
-PA28
 NoConn ~ 10550 2700
 $Comp
@@
 Wire Notes Line
 	7100 3600 7100 3950
+$Comp
+L rak4260:RAK4260 U4
+U 1 1 5DF9B993
+P 8750 2100
+F 0 "U4" H 8725 2650 59  0000 L CNB
+F 1 "RAK4260" H 9350 1700 79  0000 L CNB
+F 2 "rak4260:RAK4260-footprint_w_solder_paste" H 8650 2100 50  0001 C CNN
+F 3 "" H 8650 2100 50  0001 C CNN
+	1    8750 2100
+	1    0    0    -1
+$EndComp
 $EndSCHEMATC
